File: kicad/NadirGimbal_R2.kicad_sch (KiCad schematic)
At the start: 13 parts, among them U3 STM32G431RBT6

Commit message: docs: identify TanTaiwoo07 as project author and maintainer
Other:
- company: (none) -> TanTaiwoo07
Changed lines of the file:
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@@
 (kicad_sch (version 20230121) (generator eeschema)
   (paper "A3")
-  (title_block (title "NadirGimbal_R2 主控板") (date "2026-10-24") (rev "R2-draft") (comment1 "设计草图：打样前请在 KiCad 7+ 中运行 ERC 并按数据手册复核"))
+  (title_block (title "NadirGimbal_R2 主控板") (date "2026-10-24") (rev "R2-draft") (company "TanTaiwoo07") (comment 2 "Author: TanTaiwoo07") (comment1 "设计草图：打样前请在 KiCad 7+ 中运行 ERC 并按数据手册复核"))
 (text "NadirGimbal_R2 —— STM32G431RBT6 + 双 DRV8316R ｜ nadir 双轴（横滚+俯仰）云台主控 ｜ 原理图设计草图" (at -195 135 0) (effects (font (size 2.5 2.5) (bold) yes) (justify left)))
 (text "跨页信号全部走全局网络标签（VM/3V3/GND/3V3_ANA 及各路信号）；卫星小版（编码器/IMU）经层级端口接入。" (at -195 129 0) (effects (font (size 1.5 1.5)) (justify left)))
