File: kicad/comms.kicad_sch (KiCad schematic)
At the start: 11 parts, among them J10 SWD GH-5, J11 USB-Micro 调试, J2 MAVLINK JST-GH-4, J3 FC PWM-IN GH-3, J6 J6 SH-6, J7 J7 SH-6, J8 J8 SH-7, J9 J9 SH-7

Commit message: docs: identify TanTaiwoo07 as project author and maintainer
Other:
- company: (none) -> TanTaiwoo07
Changed lines of the file:
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@@
 (kicad_sch (version 20230121) (generator eeschema)
   (paper "A3")
-  (title_block (title "通信与传感器接口") (date "2026-10-24") (rev "R2-draft") (comment1 "设计草图：打样前请在 KiCad 7+ 中运行 ERC 并按数据手册复核"))
+  (title_block (title "通信与传感器接口") (date "2026-10-24") (rev "R2-draft") (company "TanTaiwoo07") (comment 2 "Author: TanTaiwoo07") (comment1 "设计草图：打样前请在 KiCad 7+ 中运行 ERC 并按数据手册复核"))
 (text "MAVLink v2：USART1(PB6/PB7)→J2 飞控 TELEM；调试：USART2(PA2/PA3)+J11 USB-Micro；PWM 回退输入：TIM2(PA0/PA1)→J3。" (at -180 132 0) (effects (font (size 2 2) (bold) yes) (justify left)))
 (symbol (lib_id "NGR2:Conn_01x04") (at -170 90 0) (unit 1) (exclude_from_sim no) (in_bom yes) (on_board yes) (dnp no) (fields_autoplaced yes) (property "Reference" "J2" (at -165.0 103.5 0) (effects (font (size 1.27 1.27)))) (property "Value" "MAVLINK JST-GH-4" (at -165.0 101.5 0) (effects (font (size 1.27 1.27)))) (property "Footprint" "Connector_JST:JST_GH_BM04B-GHS-TBT" (at -170 90 0) (effects (font (size 1.27 1.27)))) (pin "1")(pin "4")(pin "3")(pin "2"))
