File: kicad/drv.kicad_sch (KiCad schematic)
At the start: 36 parts, among them J4 MOTOR M1 = 横滚电机（GM3506） JST-G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, J5 MOTOR M2 = 俯仰电机（GM3506） JST-G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, U1 DRV8316R, U2 DRV8316R

Commit message: docs: identify TanTaiwoo07 as project author and maintainer
Other:
- company: (none) -> TanTaiwoo07
Changed lines of the file:
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@@
 (kicad_sch (version 20230121) (generator eeschema)
   (paper "A3")
-  (title_block (title "双路 DRV8316R 电机驱动") (date "2026-10-24") (rev "R2-draft") (comment1 "设计草图：打样前请在 KiCad 7+ 中运行 ERC 并按数据手册复核"))
+  (title_block (title "双路 DRV8316R 电机驱动") (date "2026-10-24") (rev "R2-draft") (company "TanTaiwoo07") (comment 2 "Author: TanTaiwoo07") (comment1 "设计草图：打样前请在 KiCad 7+ 中运行 ERC 并按数据手册复核"))
 (text "DRV8316R ×2，3x PWM 模式（INLx 经 0R×3 上拉至 3V3），20kHz FOC；SDO 挂共用 SPI3 MISO（nSCS 高时 Hi-Z）。" (at -180 132 0) (effects (font (size 2 2) (bold) yes) (justify left)))
 (text "每路：VM 3×100nF + bulk；CP 1uF/16V→VM；CPH-CPL 47nF；AVDD 1uF；VREF 0.1uF（0R 接 3V3）。" (at -180 126 0) (effects (font (size 1.5 1.5)) (justify left)))
