File: kicad/enc_pitch.kicad_sch (KiCad schematic)
At the start: 2 parts, among them U10 AS5048A

Commit message: docs: identify TanTaiwoo07 as project author and maintainer
Other:
- company: (none) -> TanTaiwoo07
Changed lines of the file:
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@@
 (kicad_sch (version 20230121) (generator eeschema)
   (paper "A3")
-  (title_block (title "编码器小版 - 俯仰") (date "2026-10-24") (rev "R2-draft") (comment1 "设计草图：打样前请在 KiCad 7+ 中运行 ERC 并按数据手册复核"))
+  (title_block (title "编码器小版 - 俯仰") (date "2026-10-24") (rev "R2-draft") (company "TanTaiwoo07") (comment 2 "Author: TanTaiwoo07") (comment1 "设计草图：打样前请在 KiCad 7+ 中运行 ERC 并按数据手册复核"))
 (text "AS5048A 磁编码小版（贴电机轴端）。磁钢 Ø6×2.5 径向充磁，气隙 0.5-1mm，端跳<0.05mm（定心工装保证）。" (at -165 95 0) (effects (font (size 1.5 1.5) (bold) yes) (justify left)))
 (symbol (lib_id "NGR2:AS5048A") (at -100 40 0) (unit 1) (exclude_from_sim no) (in_bom yes) (on_board yes) (dnp no) (fields_autoplaced yes) (property "Reference" "U10" (at -90.0 63.5 0) (effects (font (size 1.27 1.27)))) (property "Value" "AS5048A" (at -90.0 61.5 0) (effects (font (size 1.27 1.27)))) (property "Footprint" "Package_SO:TSSOP-14_4.4x5mm_P0.65mm" (at -100 40 0) (effects (font (size 1.27 1.27)))) (pin "1")(pin "2")(pin "3")(pin "4")(pin "5")(pin "14")(pin "13")(pin "12")(pin "11")(pin "10")(pin "9")(pin "8")(pin "7")(pin "6"))
