File: kicad/imu_base.kicad_sch (KiCad schematic)
At the start: 5 parts, among them U11 ICM-42688-P

Commit message: docs: identify TanTaiwoo07 as project author and maintainer
Other:
- company: (none) -> TanTaiwoo07
Changed lines of the file:
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@@
 (kicad_sch (version 20230121) (generator eeschema)
   (paper "A3")
-  (title_block (title "IMU 小版 - 机体侧") (date "2026-10-24") (rev "R2-draft") (comment1 "设计草图：打样前请在 KiCad 7+ 中运行 ERC 并按数据手册复核"))
+  (title_block (title "IMU 小版 - 机体侧") (date "2026-10-24") (rev "R2-draft") (company "TanTaiwoo07") (comment 2 "Author: TanTaiwoo07") (comment1 "设计草图：打样前请在 KiCad 7+ 中运行 ERC 并按数据手册复核"))
 (text "ICM-42688-P 六轴 IMU（机体侧·隔振层之下）。SPI 4 线 ≤24MHz；INT1 数据就绪中断接 MCU；ODR 建议 2-8kHz。" (at -165 95 0) (effects (font (size 1.5 1.5) (bold) yes) (justify left)))
 (symbol (lib_id "NGR2:ICM42688P") (at -100 40 0) (unit 1) (exclude_from_sim no) (in_bom yes) (on_board yes) (dnp no) (fields_autoplaced yes) (property "Reference" "U11" (at -90.0 63.5 0) (effects (font (size 1.27 1.27)))) (property "Value" "ICM-42688-P" (at -90.0 61.5 0) (effects (font (size 1.27 1.27)))) (property "Footprint" "Package_LGA:LGA-14_2.5x3mm_P0.5mm_LayoutBorder1x6y" (at -100 40 0) (effects (font (size 1.27 1.27)))) (pin "1")(pin "2")(pin "3")(pin "4")(pin "5")(pin "6")(pin "7")(pin "14")(pin "13")(pin "12")(pin "11")(pin "10")(pin "9")(pin "8"))
