File: kicad/pwr.kicad_sch (KiCad schematic)
At the start: 19 parts, among them J1 POWER_IN JST-GH-2/XT30, Q1 AO3401A 反接保护, U8 TPS54202 12V->3V3

Commit message: docs: identify TanTaiwoo07 as project author and maintainer
Other:
- company: (none) -> TanTaiwoo07
Changed lines of the file:
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@@
 (kicad_sch (version 20230121) (generator eeschema)
   (paper "A3")
-  (title_block (title "电源输入保护 + 3V3") (date "2026-10-24") (rev "R2-draft") (comment1 "设计草图：打样前请在 KiCad 7+ 中运行 ERC 并按数据手册复核"))
+  (title_block (title "电源输入保护 + 3V3") (date "2026-10-24") (rev "R2-draft") (company "TanTaiwoo07") (comment 2 "Author: TanTaiwoo07") (comment1 "设计草图：打样前请在 KiCad 7+ 中运行 ERC 并按数据手册复核"))
 (text "电源链：6S -> 独立 BEC 12V -> J1（禁止从飞控取电）-> 保险丝 -> P-MOS 反接保护 -> TVS -> VM 母线。" (at -180 130 0) (effects (font (size 2 2) (bold) yes) (justify left)))
 (text "TPS54202: 12V->3.3V/2A；3V3_ANA 经磁珠给 VDDA/VREF+。分压 100k/10k 监测 VM。" (at -180 124 0) (effects (font (size 1.5 1.5)) (justify left)))
